File: stepperCon.sch (KiCad schematic (older format))
At the start: 53 parts, among them J101 Mount_hole, J102 Mount_hole, J103 Mount_hole, J104 Mount_hole, P101 Control, P102 Phase A, P103 Phase B, P104 I2C, P105 Power, P106 Reset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

Commit message: Some comments to the code
Parts:
- Q101, Q102, Q103: symbol BSS138 -> BSS138-RESCUE-stepperCon
Changed lines of the file:
@@
 EESchema Schematic File Version 2
+LIBS:stepperCon-rescue
 LIBS:power
 LIBS:device
@@
 ENABLE_B
 $Comp
-L BSS138 Q101
+L BSS138-RESCUE-stepperCon Q101
 U 1 1 57A5214E
 P 4650 6800
@@
 $EndComp
 $Comp
-L BSS138 Q102
+L BSS138-RESCUE-stepperCon Q102
 U 1 1 57A52242
 P 4675 7350
@@
 $EndComp
 $Comp
-L BSS138 Q103
+L BSS138-RESCUE-stepperCon Q103
 U 1 1 57A6DCAA
 P 9050 1725

Commit message: First commit of working PI, with simulation Jupyter notebook.
Parts:
- removed D101: BAV99W, TO_SOT_Packages_SMD:SOT-323, symbol BAV99W
- C101, C102, C103, C104, C105, C106, C107, C108, C109, C110, C111, C112: symbol C_Small -> stepperCon-rescue:C_Small
- D102, D103: symbol Led_Small -> stepperCon-rescue:Led_Small
- J101, J102, J103, J104: symbol Mount_hole -> stepperCon-rescue:Mount_hole
- P101, P108: symbol CONN_01X06 -> stepperCon-rescue:CONN_01X06
- P102, P103, P104: symbol CONN_01X04 -> stepperCon-rescue:CONN_01X04
- P105, P106: symbol CONN_01X02 -> stepperCon-rescue:CONN_01X02
- P107: symbol CONN_U.FL -> stepperCon-rescue:CONN_U.FL
- Q101, Q102, Q103: symbol BSS138-RESCUE-stepperCon -> stepperCon-rescue:BSS138-RESCUE-stepperCon
- R101, R102, R103, R104, R105, R106, R107, R108, R109, R110, R111, R112, R113, R114, R115, R116, R117: symbol R_Small -> stepperCon-rescue:R_Small
- U101: symbol PIC18(L)F4xK22-I/PT -> stepperCon-rescue:PIC18(L)F4xK22-I_PT
- U102, U103, U104, U105: symbol MC74VHC1GT50 -> stepperCon-rescue:MC74VHC1GT50
- X101: symbol Crystal_GND3 -> stepperCon-rescue:Crystal_GND3
